File: original/QL_ROM_Cartridge_original.kicad_sch (KiCad schematic)
At the start: 6 parts, among them IC1 27C128, IC2 27C128, IC3 74LS00, J1 QL_cartridge_ROM

Commit message: Updated Original PCB
Parts:
- C1: footprint Capacitor_THT:C_Axial_L3.8mm_D2.6mm_P12.50mm_Horizontal -> 8bits:C_Axial_L3.8mm_D2.6mm_P12.50mm_Horizontal_Sinclair_Cartridge
- IC1: footprint Package_DIP:DIP-28_W15.24mm -> 8bits:DIP-28_W15.24mm_sinclair_cartridge
Connections:
- net A14: now also IC2.20 (~{CE}), IC3.4, IC3.5; no longer IC3.9
- net A15: no longer IC3.10
- net U1_CE renamed NOT_A14
- removed net U2_CE: IC2.20 (~{CE}), IC3.4, IC3.5, IC3.8
- no-connect marks 4 -> 7
Other:
- moved on the sheet: C1, C2, IC3A, IC3B, IC3C, IC3D, IC3E
